Commit message: anchor test

File: data/yumi_description/urdf/yumi.urdf (robot description, URDF)
Before this commit: robot yumi, 26 links, 25 joints
Links:
- removed link camera_link
- added link world
Joints:
- removed joint camera_joint
- added joint world_joint: type fixed, parent world, child base_link, origin xyz=0 0 0.0 rpy=0 0 0
